File: VSense.kicad_sch (KiCad schematic)
At the start: 4 parts

Commit message: added license and almost ready for prod
Parts:
- C67: Rating (none) -> 5V
- D7: footprint Diode_SMD:D_0603_1608Metric -> Diode_SMD:D_SOD-323; Rating (none) -> 1A
- R16, R17: Rating (none) -> 100mW
Changed lines of the file:
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@@
 			)
 		)
-		(property "Footprint" "Diode_SMD:D_0603_1608Metric"
+		(property "Footprint" "Diode_SMD:D_SOD-323"
 			(at 101.6 68.58 0)
 			(effects
@@
 		)
 		(property "Description" "Zener diode, filled shape"
+			(at 101.6 68.58 0)
+			(effects
+				(font
+					(size 1.27 1.27)
+				)
+				(hide yes)
+			)
+		)
+		(property "Rating" "1A"
 			(at 101.6 68.58 0)
 			(effects
@@
 			)
 		)
+		(property "Rating" "5V"
+			(at 113.03 68.58 0)
+			(effects
+				(font
+					(size 1.27 1.27)
+				)
+				(hide yes)
+			)
+		)
 		(pin "2"
 		)
@@
 			)
 		)
+		(property "Rating" "100mW"
+			(at 87.63 67.31 0)
+			(effects
+				(font
+					(size 1.27 1.27)
+				)
+				(hide yes)
+			)
+		)
 		(pin "2"
 		)
@@
 			(at 87.63 54.61 0)
 			(effects
+				(font
+					(size 1.27 1.27)
+				)
+				(hide yes)
+			)
+		)
+		(property "Rating" "100mW"
+			(at 87.63 54.61 0)
+			(effects
