File: VSupply.kicad_sch (KiCad schematic)
At the start: 11 parts, among them IC1 MP9485GN-Z

Commit message: added license and almost ready for prod
Parts:
- C61: Manufacturer_Part_Number (none) -> FS32X106K101EGG; Rating (none) -> 100V
- C62, C63, C66: Rating (none) -> 100V
- C64, C65: Rating (none) -> 6.3V
- D10: value 1.1V -> 1V; Manufacturer_Part_Number (none) -> BAV21W-AU_R1_000A1; Rating (none) -> 2A
- IC1: Height 1.7 -> (none); Manufacturer_Name Monolithic Power Systems (MPS) -> (none); Mouser Part Number 946-MP9485GN-Z -> (none); Mouser Price/Stock https://www.mouser.co.uk/ProductDetail/Monolithic-Power-Sys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 -> (none)
- L1: Rating (none) -> 1A
- R31, R32: Rating (none) -> 100mW
Changed lines of the file:
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@@
+			)
+		)
+		(property "Rating" "1A"
+			(at 119.38 62.23 0)
+			(effects
+				(font
+					(size 1.27 1.27)
+				)
+				(hide yes)
 			)
 		)
@@
 			)
 		)
+		(property "Rating" "100V"
+			(at 71.12 67.31 0)
+			(effects
+				(font
+					(size 1.27 1.27)
+				)
+				(hide yes)
+			)
+		)
 		(pin "2"
 		)
@@
 			)
 		)
+		(property "Rating" "6.3V"
+			(at 168.91 71.12 0)
+			(effects
+				(font
+					(size 1.27 1.27)
+				)
+				(hide yes)
+			)
+		)
 		(pin "2"
 		)
@@
 			)
 		)
+		(property "Rating" "100V"
+			(at 55.88 63.5 0)
+			(effects
+				(font
+					(size 1.27 1.27)
+				)
+				(hide yes)
+			)
+		)
 		(pin "2"
 		)
@@
 			)
 		)
-		(property "Value" "1.1V"
+		(property "Value" "1V"
 			(at 111.76 69.5324 90)
 			(effects
@@
 			)
 		)
+		(property "Rating" "2A"
+			(at 109.22 68.58 0)
+			(effects
+				(font
+					(size 1.27 1.27)
+				)
+				(hide yes)
+			)
+		)
+		(property "Manufacturer_Part_Number" "BAV21W-AU_R1_000A1"
+			(at 109.22 68.58 0)
+			(effects
+				(font
+					(size 1.27 1.27)
+				)
+				(hide yes)
+			)
+		)
 		(pin "1"
 		)
@@
 			)
 		)
+		(property "Rating" "100V"
+			(at 140.97 71.12 0)
+			(effects
+				(font
+					(size 1.27 1.27)
+				)
+				(hide yes)
+			)
+		)
 		(pin "2"
 		)
@@
 			)
 		)
+		(property "Rating" "100mW"
+			(at 129.54 66.04 0)
+			(effects
+				(font
+					(size 1.27 1.27)
+				)
+				(hide yes)
+			)
+		)
 		(pin "2"
 		)
@@
 			)
 		)
+		(property "Rating" "6.3V"
+			(at 154.94 71.12 0)
+			(effects
+				(font
+					(size 1.27 1.27)
+				)
+				(hide yes)
+			)
+		)
 		(pin "2"
 		)
@@
 			)
 		)
+		(property "Rating" "100mW"
+			(at 129.54 76.2 0)
+			(effects
+				(font
+					(size 1.27 1.27)
+				)
+				(hide yes)
+			)
+		)
 		(pin "2"
 		)
@@
 			)
 		)
+		(property "Rating" "100V"
+			(at 41.91 63.5 0)
+			(effects
+				(font
+					(size 1.27 1.27)
+				)
+				(hide yes)
+			)
+		)
+		(property "Manufacturer_Part_Number" "FS32X106K101EGG"
+			(at 41.91 63.5 0)
+			(effects
+				(font
+					(size 1.27 1.27)
+				)
+				(hide yes)
+			)
+		)
 		(pin "2"
 		)
@@
 			)
 		)
-		(property "Height" "1.7"
-			(at 99.06 449.53 0)
-			(effects
-				(font
-					(size 1.27 1.27)
-				)
-				(justify left top)
-				(hide yes)
-			)
-		)
-		(property "Mouser Part Number" "946-MP9485GN-Z"
-			(at 99.06 549.53 0)
-			(effects
-				(font
-					(size 1.27 1.27)
-				)
-				(justify left top)
-				(hide yes)
-			)
-		)
-		(property "Mouser Price/Stock" "https://www.mouser.co.uk/ProductDetail/Monolithic-Power-Systems-MPS/MP9485GN-Z?qs=YCa%2FAAYMW020XV52pqttNg%3D%3D"
-			(at 99.06 649.53 0)
-			(effects
-				(font
-					(size 1.27 1.27)
-				)
-				(justify left top)
-				(hide yes)
-			)
-		)
-		(property "Manufacturer_Name" "Monolithic Power Systems (MPS)"
-			(at 99.06 749.53 0)
-			(effects
-				(font
-					(size 1.27 1.27)
-				)
-				(justify left top)
-				(hide yes)
-			)
-		)
 		(property "Manufacturer_Part_Number" "MP9485GN-Z"
 			(at 99.06 849.53 0)
@@
 				(hide yes)
 			)
+		)
+		(property "Rating" ""
+			(at 77.47 54.61 0)
+			(effects
+				(font
+					(size 1.27 1.27)
+				)
+				(hide yes)
+			)
