File: VSupply.kicad_sch (KiCad schematic)
At the start: 9 parts, among them IC2 RAA2118054GP3#JA0

Commit message: Production round 1
Other:
- note added: "0-80V"
Changed lines of the file:
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@@
+		)
+	)
+	(text "0-80V"
+		(exclude_from_sim no)
+		(at 67.056 56.388 0)
+		(effects
+			(font
+				(size 1.27 1.27)
+			)
 		)
 	)

Commit message: added ESD protection
Parts:
- added D18, D19, D20: 100V, Diode_SMD:D_0603_1608Metric, symbol Device:D_TVS_Small
Connections:
- net EN: now also D20.2 (A2)
- net GND: now also D18.1 (A1), D19.1 (A1), D20.1 (A1)
- net V_{IN}: now also D18.2 (A2)
- net V_{OUT}: now also D19.2 (A2)

Commit message: added all changes from Reddit
Parts:
- removed D18, D19: 100V, Diode_SMD:D_0603_1608Metric, symbol Device:D_TVS_Small
- added D18: 6V, Diode_SMD:D_SOD-323, symbol Device:D_Zener_Filled
- added D19: 82V, Diode_SMD:D_SMA, symbol Device:D_Zener_Filled
- D20: value 100V -> 5V
Connections:
- net GND: now also D18.2 (A), D19.2 (A)
- net V_{IN}: now also D19.1 (K)
- net V_{OUT}: now also D18.1 (K)
Other:
- note added: "5V 300 mA"
- note removed: "5V 500 mA"
Changed lines of the file:
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@@
 	(wire
 		(pts
-			(xy 160.02 57.15) (xy 160.02 66.04)
-		)
-		(stroke
-			(width 0)
-			(type default)
-		)
-	)
-	(wire
-		(pts
-			(xy 45.72 68.58) (xy 45.72 80.01)
+			(xy 160.02 57.15) (xy 160.02 64.77)
+		)
+		(stroke
+			(width 0)
+			(type default)
+		)
+	)
+	(wire
+		(pts
+			(xy 160.02 72.39) (xy 160.02 78.74)
 		)
 		(stroke
@@
 	(wire
 		(pts
-			(xy 160.02 71.12) (xy 160.02 78.74)
-		)
-		(stroke
-			(width 0)
-			(type default)
-		)
-	)
-	(wire
-		(pts
 			(xy 119.38 69.85) (xy 129.54 69.85)
 		)
@@
 	(wire
 		(pts
-			(xy 45.72 57.15) (xy 45.72 63.5)
+			(xy 45.72 69.85) (xy 45.72 80.01)
+		)
+		(stroke
+			(width 0)
+			(type default)
+		)
+	)
+	(wire
+		(pts
+			(xy 45.72 57.15) (xy 45.72 62.23)
 		)
 		(stroke
@@
 		)
 	)
-	(text "5V 500 mA"
+	(text "5V 300 mA"
 		(exclude_from_sim no)
 		(at 140.716 55.88 0)
@@
 			)
 		)
-		(property "Value" "100V"
+		(property "Value" "5V"
 			(at 123.19 66.0399 90)
 			(effects
@@
 	)
 	(symbol
-		(lib_id "Device:D_TVS_Small")
-		(at 160.02 68.58 90)
-		(unit 1)
-		(exclude_from_sim no)
-		(in_bom yes)
-		(on_board yes)
-		(dnp no)
-		(fields_autoplaced yes)
-		(property "Reference" "D19"
-			(at 162.56 67.3099 90)
-			(effects
-				(font
-					(size 1.27 1.27)
-				)
-				(justify right)
-			)
-		)
-		(property "Value" "100V"
-			(at 162.56 69.8499 90)
-			(effects
-				(font
-					(size 1.27 1.27)
-				)
-				(justify right)
-			)
-		)
-		(property "Footprint" "Diode_SMD:D_0603_1608Metric"
-			(at 160.02 68.58 0)
-			(effects
-				(font
-					(size 1.27 1.27)
-				)
-				(hide yes)
-			)
-		)
-		(property "Datasheet" "~"
-			(at 160.02 68.58 0)
-			(effects
-				(font
-					(size 1.27 1.27)
-				)
-				(hide yes)
-			)
-		)
-		(property "Description" "Bidirectional transient-voltage-suppression diode, small symbol"
-			(at 160.02 68.58 0)
-			(effects
-				(font
-					(size 1.27 1.27)
-				)
-				(hide yes)
-			)
-		)
-		(property "Manufacturer_Part_Number" "ULCE1005A015FR"
-			(at 160.02 68.58 0)
-			(effects
-				(font
-					(size 1.27 1.27)
-				)
-				(hide yes)
-			)
-		)
-		(property "Source" "LCSC"
-			(at 160.02 68.58 0)
-			(effects
-				(font
-					(size 1.27 1.27)
-				)
-				(hide yes)
-			)
-		)
-		(property "Rating" "1A"
-			(at 160.02 68.58 0)
-			(effects
-				(font
-					(size 1.27 1.27)
-				)
-				(hide yes)
-			)
-		)
-		(pin "2"
-		)
-		(pin "1"
-		)
-		(instances
-			(project "OpenMD"
-				(path "/28611c8e-7644-4a1a-8c07-dc86cafc8f6c/0b9b423b-63db-4f0d-bf51-3327e1c293c5"
-					(reference "D19")
-					(unit 1)
-				)
-			)
-		)
-	)
-	(symbol
 		(lib_id "Device:C")
 		(at 147.32 68.58 0)
@@
 	)
 	(symbol
-		(lib_id "Device:D_TVS_Small")
-		(at 45.72 66.04 270)
+		(lib_id "Device:D_Zener_Filled")
+		(at 160.02 68.58 90)
 		(mirror x)
 		(unit 1)
@@
 		(dnp no)
 		(property "Reference" "D18"
-			(at 43.18 64.7699 90)
-			(effects
-				(font
-					(size 1.27 1.27)
-				)
-				(justify right)
-			)
-		)
-		(property "Value" "100V"
-			(at 43.18 67.3099 90)
-			(effects
-				(font
-					(size 1.27 1.27)
-				)
-				(justify right)
-			)
-		)
-		(property "Footprint" "Diode_SMD:D_0603_1608Metric"
-			(at 45.72 66.04 0)
+			(at 166.878 67.31 90)
+			(effects
+				(font
+					(size 1.27 1.27)
+				)
+				(justify left)
+			)
+		)
+		(property "Value" "6V"
+			(at 165.608 69.342 90)
+			(effects
+				(font
+					(size 1.27 1.27)
+				)
+				(justify left)
+			)
+		)
+		(property "Footprint" "Diode_SMD:D_SOD-323"
+			(at 160.02 68.58 0)
 			(effects
 				(font
@@
 		)
 		(property "Datasheet" "~"
-			(at 45.72 66.04 0)
-			(effects
-				(font
-					(size 1.27 1.27)
-				)
-				(hide yes)
-			)
-		)
-		(property "Description" "Bidirectional transient-voltage-suppression diode, small symbol"
-			(at 45.72 66.04 0)
-			(effects
-				(font
-					(size 1.27 1.27)
-				)
-				(hide yes)
-			)
-		)
-		(property "Manufacturer_Part_Number" "ULCE1005A015FR"
-			(at 45.72 66.04 0)
+			(at 160.02 68.58 0)
+			(effects
+				(font
+					(size 1.27 1.27)
+				)
+				(hide yes)
+			)
+		)
+		(property "Description" "Zener diode, filled shape"
+			(at 160.02 68.58 0)
+			(effects
+				(font
+					(size 1.27 1.27)
+				)
+				(hide yes)
+			)
+		)
+		(property "Rating" "1A"
+			(at 160.02 68.58 0)
+			(effects
+				(font
+					(size 1.27 1.27)
+				)
+				(hide yes)
+			)
+		)
+		(property "Manufacturer_Part_Number" "BZT52C3V3S"
+			(at 160.02 68.58 0)
 			(effects
 				(font
@@
 		)
 		(property "Source" "LCSC"
-			(at 45.72 66.04 0)
-			(effects
-				(font
-					(size 1.27 1.27)
-				)
-				(hide yes)
-			)
-		)
-		(property "Rating" "1A"
-			(at 45.72 66.04 0)
-			(effects
-				(font
-					(size 1.27 1.27)
-				)
-				(hide yes)
-			)
+			(at 160.02 68.58 0)
+			(effects
+				(font
+					(size 1.27 1.27)
+				)
+				(hide yes)
+			)
+		)
+		(pin "1"
 		)
 		(pin "2"
-		)
-		(pin "1"
 		)
 		(instances
@@
 					(unit 1)
 				)
+			)
+		)
+	)
+	(symbol
+		(lib_id "Device:D_Zener_Filled")
+		(at 45.72 66.04 270)
+		(unit 1)
+		(exclude_from_sim no)
+		(in_bom yes)
+		(on_board yes)
+		(dnp no)
+		(property "Reference" "D19"
+			(at 38.862 64.77 90)
+			(effects
+				(font
+					(size 1.27 1.27)
+				)
+				(justify left)
+			)
+		)
+		(property "Value" "82V"
+			(at 40.132 66.802 90)
+			(effects
+				(font
+					(size 1.27 1.27)
+				)
+				(justify left)
+			)
+		)
+		(property "Footprint" "Diode_SMD:D_SMA"
+			(at 45.72 66.04 0)
+			(effects
+				(font
+					(size 1.27 1.27)
+				)
+				(hide yes)
+			)
+		)
+		(property "Datasheet" "~"
+			(at 45.72 66.04 0)
+			(effects
+				(font
+					(size 1.27 1.27)
+				)
+				(hide yes)
+			)
+		)
+		(property "Description" "Zener diode, filled shape"
+			(at 45.72 66.04 0)
+			(effects
+				(font
+					(size 1.27 1.27)
+				)
+				(hide yes)
+			)
+		)
+		(property "Rating" "1A"
+			(at 45.72 66.04 0)
+			(effects
+				(font
+					(size 1.27 1.27)
+				)
+				(hide yes)
+			)
+		)
+		(property "Manufacturer_Part_Number" "BZT52C3V3S"
+			(at 45.72 66.04 0)
+			(effects
+				(font
+					(size 1.27 1.27)
+				)
+				(hide yes)
+			)
+		)
+		(property "Source" "LCSC"
+			(at 45.72 66.04 0)
+			(effects
+				(font
+					(size 1.27 1.27)
+				)
+				(hide yes)
+			)
+		)
+		(pin "1"
+		)
+		(pin "2"
+		)
+		(instances
+			(project "OpenMD"
+				(path "/28611c8e-7644-4a1a-8c07-dc86cafc8f6c/0b9b423b-63db-4f0d-bf51-3327e1c293c5"
+					(reference "D19")
+					(unit 1)
+				)

Commit message: updates to make better
Parts:
- D18: Manufacturer_Part_Number BZT52C3V3S -> MMSZ5233BS-7-F
- D19: Manufacturer_Part_Number BZT52C3V3S -> SZ4582
- D20: Manufacturer_Part_Number ULCE1005A015FR -> 0603ESDA-05N
Changed lines of the file:
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@@
 			)
 		)
-		(property "Manufacturer_Part_Number" "ULCE1005A015FR"
+		(property "Manufacturer_Part_Number" "0603ESDA-05N"
 			(at 120.65 64.77 0)
 			(effects
@@
 			)
 		)
-		(property "Manufacturer_Part_Number" "BZT52C3V3S"
+		(property "Manufacturer_Part_Number" "MMSZ5233BS-7-F"
 			(at 160.02 68.58 0)
 			(effects
@@
 			)
 		)
-		(property "Manufacturer_Part_Number" "BZT52C3V3S"
+		(property "Manufacturer_Part_Number" "SZ4582"
 			(at 45.72 66.04 0)
 			(effects

Commit message: revision 2
Parts:
- removed C11: 1uF, Capacitor_SMD:C_0805_2012Metric, symbol Device:C
- removed C63: 100nF, Capacitor_SMD:C_0603_1608Metric, symbol Device:C
- removed D10: .85V, Diode_SMD:D_SOD-123, symbol Device:D_Schottky
- removed D20: 5V, Diode_SMD:D_0603_1608Metric, symbol Device:D_TVS_Small
- removed IC2: RAA2118054GP3#JA0, Package_TO_SOT_SMD:SOT-23-5, symbol RAA2118054GP3#JA0:RAA2118054GP3#JA0
- added C11: 100nF, Capacitor_SMD:C_0402_1005Metric, symbol Device:C_Small
- added C76: 2.2nF, Capacitor_SMD:C_0402_1005Metric, symbol Device:C_Small
- added C90: 4.7uF, Capacitor_SMD:C_0402_1005Metric, symbol Device:C
- added C92: 20pF, Capacitor_SMD:C_0402_1005Metric, symbol Device:C_Small
- added R10: 72k, Resistor_SMD:R_0402_1005Metric, symbol Device:R_Small_US
- added R15: 27k, Resistor_SMD:R_0402_1005Metric, symbol Device:R_Small_US
- added R5: 240k, Resistor_SMD:R_0402_1005Metric, symbol Device:R_Small_US
- added U4: LM5164DDA, Package_SO:HSOP-8-1EP_3.9x4.9mm_P1.27mm_EP2.41x3.1mm_ThermalVias, symbol Regulator_Switching:LM5164DDA
- C1: value 1uF -> 10uF; footprint Capacitor_SMD:C_0805_2012Metric -> Capacitor_SMD:C_1210_3225Metric; Manufacturer_Part_Number HHV0805R7105K101NSLJ -> FS32X475K101EGG
- C62: value 100nF -> 220nF
- C64, C65: footprint Capacitor_SMD:C_0603_1608Metric -> Capacitor_SMD:C_0402_1005Metric
- D18: footprint Diode_SMD:D_SOD-323 -> Diode_SMD:D_SOD-882
- D19: value 82V -> 100V; footprint Diode_SMD:D_SMA -> Diode_SMD:D_SOD-123F
- L1: value 22uH -> 68uH; footprint Inductor_SMD:L_Abracon_ASPI-3012S -> Inductor_SMD:L_Abracon_ASPI-4030S
Connections:
- net EN: now also U4.3 (EN/UVLO)
- net GND: now also C11.2, C90.2, R10.2, R15.2, U4.1 (GND), U4.9 (EP)
- net SW: now also C76.2, U4.8 (SW)
- net V_{IN}: now also U4.2 (VIN)
- net V_{OUT}: now also C11.1, C90.1, C92.1, R5.1
- new net: C76.1, U4.7 (BST)
- new net: R15.1, U4.4 (RON)
- new net FB: C92.2, R10.1, R5.2, U4.5 (FB)
- no-connect marks 0 -> 1
Other:
- note added: "0-100V"
- note added: "5.2V 300mA"
- note added: "Can be any LM561*"
- note added: "f_{SW} = (V_{OUT} * 2500) / R_{ON}"
- note added: "f_{SW} = ~500kHz"
- note added: "t_{ONMIN} = 100ns"
- note added: "t_{ON} (us) = R_{ON} / (V_{IN} * 2500)"
- note removed: "0-80V"
- note removed: "5V 300 mA"
- moved on the sheet: C62, C64, C65, D18, D19, L1

Commit message: next generation
Parts:
- C62: value 220nF -> 100nF
Changed lines of the file:
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@@
 			)
 		)
-		(property "Value" "220nF"
+		(property "Value" "100nF"
 			(at 50.8 60.9599 0)
 			(effects

Commit message: added more capacitance
Parts:
- C1: footprint Capacitor_SMD:C_1210_3225Metric -> OpenMD:C_1210_3225Metric; symbol Device:C -> OpenMD:C
- C11, C76, C92: footprint Capacitor_SMD:C_0402_1005Metric -> OpenMD:C_0402_1005Metric; symbol Device:C_Small -> OpenMD:C_Small
- C62: footprint Capacitor_SMD:C_0603_1608Metric -> OpenMD:C_0603_1608Metric; symbol Device:C -> OpenMD:C
- C64, C65, C90: footprint Capacitor_SMD:C_0402_1005Metric -> OpenMD:C_0402_1005Metric; symbol Device:C -> OpenMD:C
- D18: footprint Diode_SMD:D_SOD-882 -> OpenMD:D_SOD-882; symbol Device:D_Zener_Filled -> OpenMD:D_Zener_Filled
- D19: footprint Diode_SMD:D_SOD-123F -> OpenMD:D_SOD-123F; symbol Device:D_Zener_Filled -> OpenMD:D_Zener_Filled
- L1: footprint Inductor_SMD:L_Abracon_ASPI-4030S -> OpenMD:L_Abracon_ASPI-4030S; symbol Device:L -> OpenMD:L
- R10, R15, R5: footprint Resistor_SMD:R_0402_1005Metric -> OpenMD:R_0402_1005Metric; symbol Device:R_Small_US -> OpenMD:R_Small_US
- U4: footprint Package_SO:HSOP-8-1EP_3.9x4.9mm_P1.27mm_EP2.41x3.1mm_ThermalVias -> OpenMD:HSOP-8-1EP_3.9x4.9mm_P1.27mm_EP2.41x3.1mm_ThermalVias; symbol Regulator_Switching:LM5164DDA -> OpenMD:LM5164DDA
Changed lines of the file:
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@@
 	(title_block
 		(title "Gate Driver Voltage Supply")
-		(date "2024-05-19")
-		(rev "1")
+		(date "2024-12-19")
+		(rev "1.1")
 		(company "Crab Labs")
 		(comment 1 "Author: Orion Serup")
@@
 	)
 	(symbol
-		(lib_id "Device:C_Small")
+		(lib_id "OpenMD:C_Small")
 		(at 123.19 59.69 0)
 		(unit 1)
@@
 			)
 		)
-		(property "Footprint" "Capacitor_SMD:C_0402_1005Metric"
+		(property "Footprint" "OpenMD:C_0402_1005Metric"
 			(at 123.19 59.69 0)
 			(effects
@@
 	)
 	(symbol
-		(lib_id "Device:C_Small")
+		(lib_id "OpenMD:C_Small")
 		(at 140.97 63.5 0)
 		(mirror y)
@@
 			)
 		)
-		(property "Footprint" "Capacitor_SMD:C_0402_1005Metric"
+		(property "Footprint" "OpenMD:C_0402_1005Metric"
 			(at 140.97 63.5 0)
 			(effects
@@
 	)
 	(symbol
-		(lib_id "Device:L")
+		(lib_id "OpenMD:L")
 		(at 105.41 57.15 90)
 		(unit 1)
@@
 			)
 		)
-		(property "Footprint" "Inductor_SMD:L_Abracon_ASPI-4030S"
+		(property "Footprint" "OpenMD:L_Abracon_ASPI-4030S"
 			(at 105.41 57.15 0)
 			(effects
@@
 	)
 	(symbol
-		(lib_id "Device:C")
+		(lib_id "OpenMD:C")
 		(at 157.48 63.5 0)
 		(unit 1)
@@
 			)
 		)
-		(property "Footprint" "Capacitor_SMD:C_0402_1005Metric"
+		(property "Footprint" "OpenMD:C_0402_1005Metric"
 			(at 158.4452 67.31 0)
 			(effects
@@
 	)
 	(symbol
-		(lib_id "Device:C_Small")
+		(lib_id "OpenMD:C_Small")
 		(at 91.44 54.61 0)
 		(unit 1)
@@
 			)
 		)
-		(property "Footprint" "Capacitor_SMD:C_0402_1005Metric"
+		(property "Footprint" "OpenMD:C_0402_1005Metric"
 			(at 91.44 54.61 0)
 			(effects
@@
 	)
 	(symbol
-		(lib_id "Device:C")
+		(lib_id "OpenMD:C")
 		(at 46.99 59.69 0)
 		(unit 1)
@@
 			)
 		)
-		(property "Footprint" "Capacitor_SMD:C_0603_1608Metric"
+		(property "Footprint" "OpenMD:C_0603_1608Metric"
 			(at 47.9552 63.5 0)
 			(effects
@@
 	)
 	(symbol
-		(lib_id "Device:D_Zener_Filled")
+		(lib_id "OpenMD:D_Zener_Filled")
 		(at 179.07 60.96 90)
 		(mirror x)
@@
 			)
 		)
-		(property "Footprint" "Diode_SMD:D_SOD-882"
+		(property "Footprint" "OpenMD:D_SOD-882"
 			(at 179.07 60.96 0)
 			(effects
@@
 	)
 	(symbol
-		(lib_id "Regulator_Switching:LM5164DDA")
+		(lib_id "OpenMD:LM5164DDA")
 		(at 74.93 59.69 0)
 		(unit 1)
@@
 			)
 		)
-		(property "Footprint" "Package_SO:HSOP-8-1EP_3.9x4.9mm_P1.27mm_EP2.41x3.1mm_ThermalVias"
+		(property "Footprint" "OpenMD:HSOP-8-1EP_3.9x4.9mm_P1.27mm_EP2.41x3.1mm_ThermalVias"
 			(at 76.2 71.12 0)
 			(effects
@@
 	)
 	(symbol
-		(lib_id "Device:C")
+		(lib_id "OpenMD:C")
 		(at 36.83 62.23 0)
 		(unit 1)
@@
 			)
 		)
-		(property "Footprint" "Capacitor_SMD:C_1210_3225Metric"
+		(property "Footprint" "OpenMD:C_1210_3225Metric"
 			(at 37.7952 66.04 0)
 			(effects
@@
 	)
 	(symbol
-		(lib_id "Device:R_Small_US")
+		(lib_id "OpenMD:R_Small_US")
 		(at 60.96 69.85 0)
 		(mirror y)
@@
 			)
 		)
-		(property "Footprint" "Resistor_SMD:R_0402_1005Metric"
+		(property "Footprint" "OpenMD:R_0402_1005Metric"
 			(at 60.96 69.85 0)
 			(effects
@@
 	)
 	(symbol
-		(lib_id "Device:D_Zener_Filled")
+		(lib_id "OpenMD:D_Zener_Filled")
 		(at 29.21 60.96 270)
 		(unit 1)
@@
 			)
 		)
-		(property "Footprint" "Diode_SMD:D_SOD-123F"
+		(property "Footprint" "OpenMD:D_SOD-123F"
 			(at 29.21 60.96 0)
 			(effects
@@
 	)
 	(symbol
-		(lib_id "Device:R_Small_US")
+		(lib_id "OpenMD:R_Small_US")
 		(at 111.76 69.85 0)
 		(unit 1)
@@
 			)
 		)
-		(property "Footprint" "Resistor_SMD:R_0402_1005Metric"
+		(property "Footprint" "OpenMD:R_0402_1005Metric"
 			(at 111.76 69.85 0)
 			(effects
@@
 	)
 	(symbol
-		(lib_id "Device:R_Small_US")
+		(lib_id "OpenMD:R_Small_US")
 		(at 111.76 59.69 0)
 		(unit 1)
@@
 			)
 		)
-		(property "Footprint" "Resistor_SMD:R_0402_1005Metric"
+		(property "Footprint" "OpenMD:R_0402_1005Metric"
 			(at 111.76 59.69 0)
 			(effects
@@
 	)
 	(symbol
-		(lib_id "Device:C")
+		(lib_id "OpenMD:C")
 		(at 168.91 63.5 0)
 		(unit 1)
@@
 			)
 		)
-		(property "Footprint" "Capacitor_SMD:C_0402_1005Metric"
+		(property "Footprint" "OpenMD:C_0402_1005Metric"
 			(at 169.8752 67.31 0)
 			(effects
@@
 	)
 	(symbol
-		(lib_id "Device:C")
+		(lib_id "OpenMD:C")
 		(at 152.4 63.5 0)
 		(mirror y)
@@
 			)
 		)
-		(property "Footprint" "Capacitor_SMD:C_0402_1005Metric"
+		(property "Footprint" "OpenMD:C_0402_1005Metric"
 			(at 151.4348 67.31 0)
 			(effects
