File: OpenMD.kicad_sch (KiCad schematic)
At the start: 18 parts, among them J1 GND, J2 Digital, J3 Analog, J4 Sensors, J5 A, J6 B, J7 C, J8 V_{BATT}

Commit message: first fab run
Parts:
- added C76, C77: 100nF, Capacitor_SMD:C_0603_1608Metric, symbol Device:C
- added H6: M2, MountingHole:MountingHole_2.2mm_M2, symbol Mechanical:MountingHole
- added R33, R34: 10k, Resistor_SMD:R_0603_1608Metric, symbol Device:R_US
- added SYM1: Logo_Open_Hardware_Large, Symbol:OSHW-Symbol_8.9x8mm_SilkScreen, symbol Graphic:Logo_Open_Hardware_Large
- added TH1, TH2: 10k, Resistor_SMD:R_0603_1608Metric, symbol Device:Thermistor_NTC_US
- FID1, FID2, FID3, FID4, FID5, FID6: Manufacturer_Part_Number (none) -> N/A; Source (none) -> N/A
- H1, H2, H3, H4: value MountingHole_Pad -> M3; Manufacturer_Part_Number (none) -> N/A; Source (none) -> N/A
- J1, J5, J6, J7, J8: Manufacturer_Part_Number (none) -> AMT0440005TH0000G; Rating (none) -> 80A; Source (none) -> Digikey
- J2, J3: Manufacturer_Part_Number (none) -> SM12B-SRSS-TB(LF)(SN); Rating (none) -> 1A; Source (none) -> LCSC
- J4: footprint Connector_JST:JST_PH_S6B-PH-SM4-TB_1x06-1MP_P2.00mm_Horizontal -> Connector_JST:JST_PH_S6B-PH-K_1x06_P2.00mm_Horizontal; Manufacturer_Part_Number (none) -> S6B-PH-K-S(LF)(SN); Rating (none) -> 1A; Source (none) -> LCSC
Connections:
- net DRV_I_SENSE.A is gone; now on net V_SENSE.A: J3.8 (Pin_8)
- net DRV_I_SENSE.B is gone; now on net V_SENSE.B: J3.9 (Pin_9)
- net DRV_I_SENSE.C is gone; now on net V_SENSE.C: J3.10 (Pin_10)
- net GND: now also J3.2 (Pin_2), J3.7 (Pin_7), J4.1 (Pin_1), C76.2, C77.2, TH1.2, TH2.2; no longer J4.6 (Pin_6)
- net HALL.A: now also J4.4 (Pin_4); no longer J4.3 (Pin_3)
- net HALL.B: now also J4.3 (Pin_3); no longer J4.4 (Pin_4)
- net HALL.C: now also J4.2 (Pin_2); no longer J4.5 (Pin_5)
- net I_SENSE.A: now also J3.3 (Pin_3); no longer J3.2 (Pin_2)
- net I_SENSE.B: now also J3.4 (Pin_4); no longer J3.3 (Pin_3)
- net I_SENSE.C: now also J3.5 (Pin_5); no longer J3.4 (Pin_4)
- net M_TEMP_SENSE: now also J4.5 (Pin_5), C76.1, R33.2, TH2.1; no longer J4.2 (Pin_2)
- net V_SENSE.A: no longer J3.5 (Pin_5)
- net V_SENSE.B: no longer J3.6 (Pin_6)
- net V_SENSE.C: no longer J3.7 (Pin_7)
- net V_{ANA}: now also R33.1, R34.1
- net V_{DIG}: now also J4.6 (Pin_6); no longer J4.1 (Pin_1)
- new net DRV_TEMP_SENSE: C77.1, J3.6 (Pin_6), R34.2, TH1.1
Other:
- removed sheet Driver Current Sensors
- sheet Drivers ports: added none; removed I_SENSE{PHASES}
- note added: "Theoretical System Ratings: V_{BATT}: 6-80V I_{BATT}: 0-73A RMS P_{MAX}: 4 kW"
- title: (none) -> 3 Phase Motor Driver
- moved on the sheet: J4, J5, J6, J7
