File: VoltageSensors.kicad_sch (KiCad schematic)
At the start: 12 parts

Commit message: adjusted according to Reddit feedback
Still needs TVS adjusted
Parts:
- D7, D8, D9: value 3.3V -> 3.6V
Changed lines of the file:
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@@
 			)
 		)
-		(property "Value" "3.3V"
+		(property "Value" "3.6V"
 			(at 147.32 67.3099 90)
 			(effects
@@
 			)
 		)
-		(property "Value" "3.3V"
+		(property "Value" "3.6V"
 			(at 147.32 102.8699 90)
 			(effects
@@
 			)
 		)
-		(property "Value" "3.3V"
+		(property "Value" "3.6V"
 			(at 147.32 137.1599 90)
 			(effects
