File: VoltageSensors.kicad_sch (KiCad schematic)
At the start: 12 parts

Commit message: updates to make better
Parts:
- D7, D8, D9: value 3.6V -> 3.3V
Changed lines of the file:
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@@
 			)
 		)
-		(property "Value" "3.6V"
+		(property "Value" "3.3V"
 			(at 147.32 67.3099 90)
 			(effects
@@
 			)
 		)
-		(property "Value" "3.6V"
+		(property "Value" "3.3V"
 			(at 147.32 102.8699 90)
 			(effects
@@
 			)
 		)
-		(property "Value" "3.6V"
+		(property "Value" "3.3V"
 			(at 147.32 137.1599 90)
 			(effects

Commit message: revision 2
Parts:
- removed D7, D8, D9: 3.3V, Diode_SMD:D_SOD-323, symbol Device:D_Zener_Filled
- C67, C68, C69: footprint Capacitor_SMD:C_0603_1608Metric -> Capacitor_SMD:C_0402_1005Metric
- R16, R17, R18, R19, R20, R21: footprint Resistor_SMD:R_0603_1608Metric -> Resistor_SMD:R_0402_1005Metric
Other:
- note removed: "Over Voltage Protection"
- moved on the sheet: C67, C68, C69
