File: Drivers.kicad_sch (KiCad schematic)
At the start: 41 parts

Commit message: added license and almost ready for prod
Parts:
- C1, C10, C11, C12, C13, C14, C15, C16, C17, C18, C19, C2, C20, C21, C22, C23, C24, C25, C26, C27, C3, C4, C5, C6, C7, C77, C78, C79, C8, C80, C81, C82, C83, C84, C85, C86, C87, C88, C89, C9, C91: Manufacturer_Part_Number (none) -> FS32X106K101EGG; Rating (none) -> 100V

Commit message: first fab run
Parts:
- removed C1, C10, C11, C13, C14, C16, C17, C20, C22, C25, C4, C5, C77, C83, C84, C85: 10uF, Capacitor_SMD:C_1210_3225Metric, symbol Device:C
- C12, C15, C18, C19, C2, C21, C23, C24, C26, C27, C3, C6, C7, C78, C79, C8, C80, C81, C82, C86, C87, C88, C89, C9, C91: value 10uF -> 4.7uF; Manufacturer_Part_Number FS32X106K101EGG -> FS32X475K101EGG; Source (none) -> LCSC
Other:
- sheet Phase Driver A ports: added none; removed I_SENSE
- sheet Phase Driver B ports: added none; removed I_SENSE
- sheet Phase Driver C ports: added none; removed I_SENSE
- note added: "Bulk Capacitors"
- moved on the sheet: C12, C15, C18, C2, C21, C23, C24, C26, C27, C3, C6, C78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

Commit message: updates to make better
Parts:
- C12, C15, C18, C19, C2, C21, C23, C24, C26, C27, C3, C6, C7, C78, C79, C8, C80, C81, C82, C86, C87, C88, C89, C9, C91: value 4.7uF -> 10uF
Changed lines of the file:
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@@
 			)
 		)
-		(property "Value" "4.7uF"
+		(property "Value" "10uF"
 			(at 134.62 93.9799 0)
 			(effects
@@
 			)
 		)
-		(property "Value" "4.7uF"
+		(property "Value" "10uF"
 			(at 59.69 43.1799 0)
 			(effects
@@
 			)
 		)
-		(property "Value" "4.7uF"
+		(property "Value" "10uF"
 			(at 109.22 68.5799 0)
 			(effects
@@
 			)
 		)
-		(property "Value" "4.7uF"
+		(property "Value" "10uF"
 			(at 109.22 93.9799 0)
 			(effects
@@
 			)
 		)
-		(property "Value" "4.7uF"
+		(property "Value" "10uF"
 			(at 96.52 68.5799 0)
 			(effects
@@
 			)
 		)
-		(property "Value" "4.7uF"
+		(property "Value" "10uF"
 			(at 146.05 68.5799 0)
 			(effects
@@
 			)
 		)
-		(property "Value" "4.7uF"
+		(property "Value" "10uF"
 			(at 121.92 68.5799 0)
 			(effects
@@
 			)
 		)
-		(property "Value" "4.7uF"
+		(property "Value" "10uF"
 			(at 96.52 43.1799 0)
 			(effects
@@
 			)
 		)
-		(property "Value" "4.7uF"
+		(property "Value" "10uF"
 			(at 83.82 43.1799 0)
 			(effects
@@
 			)
 		)
-		(property "Value" "4.7uF"
+		(property "Value" "10uF"
 			(at 133.35 68.5799 0)
 			(effects
@@
 			)
 		)
-		(property "Value" "4.7uF"
+		(property "Value" "10uF"
 			(at 59.69 68.5799 0)
 			(effects
@@
 			)
 		)
-		(property "Value" "4.7uF"
+		(property "Value" "10uF"
 			(at 121.92 93.9799 0)
 			(effects
@@
 			)
 		)
-		(property "Value" "4.7uF"
+		(property "Value" "10uF"
 			(at 85.09 93.9799 0)
 			(effects
@@
 			)
 		)
-		(property "Value" "4.7uF"
+		(property "Value" "10uF"
 			(at 109.22 43.1799 0)
 			(effects
@@
 			)
 		)
-		(property "Value" "4.7uF"
+		(property "Value" "10uF"
 			(at 72.39 43.1799 0)
 			(effects
@@
 			)
 		)
-		(property "Value" "4.7uF"
+		(property "Value" "10uF"
 			(at 72.39 68.5799 0)
 			(effects
@@
 			)
 		)
-		(property "Value" "4.7uF"
+		(property "Value" "10uF"
 			(at 158.75 68.5799 0)
 			(effects
@@
 			)
 		)
-		(property "Value" "4.7uF"
+		(property "Value" "10uF"
 			(at 133.35 43.1799 0)
 			(effects
@@
 			)
 		)
-		(property "Value" "4.7uF"
+		(property "Value" "10uF"
 			(at 83.82 68.5799 0)
 			(effects
@@
 			)
 		)
-		(property "Value" "4.7uF"
+		(property "Value" "10uF"
 			(at 60.96 93.9799 0)
 			(effects
@@
 			)
 		)
-		(property "Value" "4.7uF"
+		(property "Value" "10uF"
 			(at 96.52 93.9799 0)
 			(effects
@@
 			)
 		)
-		(property "Value" "4.7uF"
+		(property "Value" "10uF"
 			(at 158.75 43.1799 0)
 			(effects
@@
 			)
 		)
-		(property "Value" "4.7uF"
+		(property "Value" "10uF"
 			(at 121.92 43.1799 0)
 			(effects
@@
 			)
 		)
-		(property "Value" "4.7uF"
+		(property "Value" "10uF"
 			(at 146.05 43.1799 0)
 			(effects
@@
 			)
 		)
-		(property "Value" "4.7uF"
+		(property "Value" "10uF"
 			(at 72.39 93.9799 0)
 			(effects

Commit message: next generation
Parts:
- added C100, C101, C102, C103, C93, C94, C98, C99: 10uF, Capacitor_SMD:C_1210_3225Metric, symbol Device:C
Connections:
- net GND: now also C100.2, C101.2, C102.2, C103.2, C93.2, C94.2, C98.2, C99.2
- net V_{MOTOR}: now also C100.1, C101.1, C102.1, C103.1, C93.1, C94.1, C98.1, C99.1

Commit message: added more capacitance
Parts:
- added C104, C105, C106, C107, C108: 10uF, OpenMD:C_1210_3225Metric, symbol OpenMD:C
- C100, C101, C102, C103, C12, C15, C18, C19, C2, C21, C23, C24, C26, C27, C3, C6, C7, C78, C79, C8, C80, C81, C82, C86, C87, C88, C89, C9, C91, C93, C94, C98, C99: footprint Capacitor_SMD:C_1210_3225Metric -> OpenMD:C_1210_3225Metric; symbol Device:C -> OpenMD:C
Connections:
- net GND: now also C104.2, C105.2, C106.2, C107.2, C108.2
- net V_{MOTOR}: now also C104.1, C105.1, C106.1, C107.1, C108.1
