File: ISense.kicad_sch (KiCad schematic)
At the start: 8 parts, among them U8 INA241A2

Commit message: revision 2
Parts:
- removed D21: 3.3V, Diode_SMD:D_SOD-323, symbol Device:D_Zener_Filled
- removed D24: 100V, Diode_SMD:D_0603_1608Metric, symbol Device:D_TVS_Small
- added D7: 100V, Diode_SMD:D_SOD-123F, symbol Device:D_Zener_Small_Filled
- C47, C49: footprint Capacitor_SMD:C_0603_1608Metric -> Capacitor_SMD:C_0402_1005Metric
- R22, R24: footprint Resistor_SMD:R_0603_1608Metric -> Resistor_SMD:R_0402_1005Metric
- R23: value .3m -> .5m
Connections:
- net GND: now also D7.2 (A)
- net I_{OUT}: now also D7.1 (K)
Other:
- note added: "Gain = 20"
- note added: "I_{MAX} = 165A, I_{MIN} = -165A, V_{DDA} = 3.3V, V_{REF} = 1.65"
- note added: "V_{SENSE} = V_{REF} + I_{SHUNT} * .01"
- note removed: "Gain = 50"
- note removed: "I_{MAX} = 110A, I_{MIN} = -110A, V_{DDA} = 3.3V, V_{REF} = 1.65"
- note removed: "V_{SENSE} = V_{REF} + I_{SHUNT} * .015"
Changed lines of the file:
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@@
-	)
-	(junction
-		(at 115.57 91.44)
-		(diameter 0)
-		(color 0 0 0 0)
 	)
 	(junction
@@
 	(wire
 		(pts
-			(xy 115.57 91.44) (xy 118.11 91.44)
+			(xy 107.95 91.44) (xy 118.11 91.44)
 		)
 		(stroke
@@
 	(wire
 		(pts
-			(xy 107.95 91.44) (xy 115.57 91.44)
-		)
-		(stroke
-			(width 0)
-			(type default)
-		)
-	)
-	(wire
-		(pts
-			(xy 114.3 101.6) (xy 115.57 100.33)
-		)
-		(stroke
-			(width 0)
-			(type default)
-		)
-	)
-	(wire
-		(pts
-			(xy 115.57 99.06) (xy 115.57 100.33)
-		)
-		(stroke
-			(width 0)
-			(type default)
-		)
-	)
-	(wire
-		(pts
 			(xy 81.28 92.71) (xy 86.36 92.71)
 		)
@@
 		(pts
 			(xy 104.14 68.58) (xy 104.14 73.66)
-		)
-		(stroke
-			(width 0)
-			(type default)
-		)
-	)
-	(wire
-		(pts
-			(xy 113.03 101.6) (xy 114.3 101.6)
 		)
 		(stroke
@@
 		)
 	)
-	(text "V_{SENSE} = V_{REF} + I_{SHUNT} * .015"
+	(text "V_{SENSE} = V_{REF} + I_{SHUNT} * .01"
 		(exclude_from_sim no)
 		(at 149.098 91.186 0)
@@
 		)
 	)
-	(text "Gain = 50\n"
+	(text "Gain = 20\n"
 		(exclude_from_sim no)
 		(at 115.824 74.168 0)
@@
 		)
 	)
-	(text "I_{MAX} = 110A, I_{MIN} = -110A, V_{DDA} = 3.3V, V_{REF} = 1.65"
+	(text "I_{MAX} = 165A, I_{MIN} = -165A, V_{DDA} = 3.3V, V_{REF} = 1.65"
 		(exclude_from_sim no)
 		(at 159.004 93.726 0)
@@
 		)
 	)
-	(hierarchical_label "GND"
-		(shape passive)
-		(at 113.03 101.6 180)
-		(fields_autoplaced yes)
-		(effects
-			(font
-				(size 1.27 1.27)
-			)
-			(justify right)
-		)
-	)
 	(hierarchical_label "SENSE"
 		(shape output)
@@
 			)
 			(justify left)
-		)
-	)
-	(symbol
-		(lib_id "Device:D_Zener_Filled")
-		(at 115.57 95.25 90)
-		(mirror x)
-		(unit 1)
-		(exclude_from_sim no)
-		(in_bom yes)
-		(on_board yes)
-		(dnp no)
-		(property "Reference" "D21"
-			(at 122.428 93.98 90)
-			(effects
-				(font
-					(size 1.27 1.27)
-				)
-				(justify left)
-			)
-		)
-		(property "Value" "3.3V"
-			(at 122.936 96.012 90)
-			(effects
-				(font
-					(size 1.27 1.27)
-				)
-				(justify left)
-			)
-		)
-		(property "Footprint" "Diode_SMD:D_SOD-323"
-			(at 115.57 95.25 0)
-			(effects
-				(font
-					(size 1.27 1.27)
-				)
-				(hide yes)
-			)
-		)
-		(property "Datasheet" "~"
-			(at 115.57 95.25 0)
-			(effects
-				(font
-					(size 1.27 1.27)
-				)
-				(hide yes)
-			)
-		)
-		(property "Description" "Zener diode, filled shape"
-			(at 115.57 95.25 0)
-			(effects
-				(font
-					(size 1.27 1.27)
-				)
-				(hide yes)
-			)
-		)
-		(property "Rating" "1A"
-			(at 115.57 95.25 0)
-			(effects
-				(font
-					(size 1.27 1.27)
-				)
-				(hide yes)
-			)
-		)
-		(property "Manufacturer_Part_Number" "BZT52C3V3S"
-			(at 115.57 95.25 0)
-			(effects
-				(font
-					(size 1.27 1.27)
-				)
-				(hide yes)
-			)
-		)
-		(property "Source" "LCSC"
-			(at 115.57 95.25 0)
-			(effects
-				(font
-					(size 1.27 1.27)
-				)
-				(hide yes)
-			)
-		)
-		(pin "1"
-		)
-		(pin "2"
-		)
-		(instances
-			(project "OpenMD"
-				(path "/28611c8e-7644-4a1a-8c07-dc86cafc8f6c/2a00e860-f835-428e-8d60-1f81dad8d039/333c1edc-8103-4690-800d-12fcc828edaf"
-					(reference "D21")
-					(unit 1)
-				)
-				(path "/28611c8e-7644-4a1a-8c07-dc86cafc8f6c/2a00e860-f835-428e-8d60-1f81dad8d039/7e19f11a-277e-4650-9782-9c7c2d21b0fd"
-					(reference "D22")
-					(unit 1)
-				)
-				(path "/28611c8e-7644-4a1a-8c07-dc86cafc8f6c/2a00e860-f835-428e-8d60-1f81dad8d039/c7f7d708-2dea-4049-a8c4-f9d7592eff53"
-					(reference "D23")
-					(unit 1)
-				)
-			)
-		)
-	)
-	(symbol
-		(lib_id "Device:D_TVS_Small")
-		(at 125.73 44.45 270)
-		(mirror x)
-		(unit 1)
-		(exclude_from_sim no)
-		(in_bom yes)
-		(on_board yes)
-		(dnp no)
-		(property "Reference" "D24"
-			(at 123.19 43.1799 90)
-			(effects
-				(font
-					(size 1.27 1.27)
-				)
-				(justify right)
-			)
-		)
-		(property "Value" "100V"
-			(at 123.19 45.7199 90)
-			(effects
-				(font
-					(size 1.27 1.27)
-				)
-				(justify right)
-			)
-		)
-		(property "Footprint" "Diode_SMD:D_0603_1608Metric"
-			(at 125.73 44.45 0)
-			(effects
-				(font
-					(size 1.27 1.27)
-				)
-				(hide yes)
-			)
-		)
-		(property "Datasheet" "~"
-			(at 125.73 44.45 0)
-			(effects
-				(font
-					(size 1.27 1.27)
-				)
-				(hide yes)
-			)
-		)
-		(property "Description" "Bidirectional transient-voltage-suppression diode, small symbol"
-			(at 125.73 44.45 0)
-			(effects
-				(font
-					(size 1.27 1.27)
-				)
-				(hide yes)
-			)
-		)
-		(property "Manufacturer_Part_Number" "ULCE1005A015FR"
-			(at 125.73 44.45 0)
-			(effects
-				(font
-					(size 1.27 1.27)
-				)
-				(hide yes)
-			)
-		)
-		(property "Source" "LCSC"
-			(at 125.73 44.45 0)
-			(effects
-				(font
-					(size 1.27 1.27)
-				)
-				(hide yes)
-			)
-		)
-		(property "Rating" "1A"
-			(at 125.73 44.45 0)
-			(effects
-				(font
-					(size 1.27 1.27)
-				)
-				(hide yes)
-			)
-		)
-		(pin "2"
-		)
-		(pin "1"
-		)
-		(instances
-			(project "OpenMD"
-				(path "/28611c8e-7644-4a1a-8c07-dc86cafc8f6c/2a00e860-f835-428e-8d60-1f81dad8d039/333c1edc-8103-4690-800d-12fcc828edaf"
-					(reference "D24")
-					(unit 1)
-				)
-				(path "/28611c8e-7644-4a1a-8c07-dc86cafc8f6c/2a00e860-f835-428e-8d60-1f81dad8d039/7e19f11a-277e-4650-9782-9c7c2d21b0fd"
-					(reference "D25")
-					(unit 1)
-				)
-				(path "/28611c8e-7644-4a1a-8c07-dc86cafc8f6c/2a00e860-f835-428e-8d60-1f81dad8d039/c7f7d708-2dea-4049-a8c4-f9d7592eff53"
-					(reference "D26")
-					(unit 1)
-				)
-			)
 		)
 	)
@@
 			)
 		)
-		(property "Footprint" "Capacitor_SMD:C_0603_1608Metric"
+		(property "Footprint" "Capacitor_SMD:C_0402_1005Metric"
 			(at 106.68 62.23 0)
 			(effects
@@
 			)
 		)
-		(property "Footprint" "Resistor_SMD:R_0603_1608Metric"
+		(property "Footprint" "Resistor_SMD:R_0402_1005Metric"
 			(at 101.6 55.88 0)
 			(effects
@@
 			)
 		)
-		(property "Footprint" "Capacitor_SMD:C_0603_1608Metric"
+		(property "Footprint" "Capacitor_SMD:C_0402_1005Metric"
 			(at 87.63 83.82 0)
 			(effects
@@
 			)
 		)
-		(property "Value" ".3m"
+		(property "Value" ".5m"
 			(at 106.68 36.83 90)
 			(effects
@@
 			)
 		)
-		(property "Footprint" "Resistor_SMD:R_0603_1608Metric"
+		(property "Footprint" "Resistor_SMD:R_0402_1005Metric"
 			(at 111.76 55.88 0)
 			(effects
@@
 					(unit 1)
 				)
+			)
+		)
+	)
+	(symbol
+		(lib_id "Device:D_Zener_Small_Filled")
+		(at 125.73 44.45 270)
+		(unit 1)
+		(exclude_from_sim no)
+		(in_bom yes)
+		(on_board yes)
+		(dnp no)
+		(fields_autoplaced yes)
+		(property "Reference" "D7"
+			(at 128.27 43.1799 90)
+			(effects
+				(font
+					(size 1.27 1.27)
+				)
+				(justify left)
+			)
+		)
+		(property "Value" "100V"
+			(at 128.27 45.7199 90)
+			(effects
+				(font
+					(size 1.27 1.27)
+				)
+				(justify left)
+			)
+		)
+		(property "Footprint" "Diode_SMD:D_SOD-123F"
+			(at 125.73 44.45 90)
+			(effects
+				(font
+					(size 1.27 1.27)
+				)
+				(hide yes)
+			)
+		)
+		(property "Datasheet" "~"
+			(at 125.73 44.45 90)
+			(effects
+				(font
+					(size 1.27 1.27)
+				)
+				(hide yes)
+			)
+		)
+		(property "Description" "Zener diode, small symbol, filled shape"
+			(at 125.73 44.45 0)
+			(effects
+				(font
+					(size 1.27 1.27)
+				)
+				(hide yes)
+			)
+		)
+		(pin "1"
+		)
+		(pin "2"
+		)
+		(instances
+			(project ""
+				(path "/28611c8e-7644-4a1a-8c07-dc86cafc8f6c/2a00e860-f835-428e-8d60-1f81dad8d039/333c1edc-8103-4690-800d-12fcc828edaf"
+					(reference "D7")
+					(unit 1)
+				)
+				(path "/28611c8e-7644-4a1a-8c07-dc86cafc8f6c/2a00e860-f835-428e-8d60-1f81dad8d039/7e19f11a-277e-4650-9782-9c7c2d21b0fd"
+					(reference "D8")
+					(unit 1)
+				)
+				(path "/28611c8e-7644-4a1a-8c07-dc86cafc8f6c/2a00e860-f835-428e-8d60-1f81dad8d039/c7f7d708-2dea-4049-a8c4-f9d7592eff53"
+					(reference "D9")
+					(unit 1)
+				)

Commit message: added more capacitance
Parts:
- C47, C49: footprint Capacitor_SMD:C_0402_1005Metric -> OpenMD:C_0402_1005Metric; symbol Device:C_Small -> OpenMD:C_Small
- D7: footprint Diode_SMD:D_SOD-123F -> OpenMD:D_SOD-123F; symbol Device:D_Zener_Small_Filled -> OpenMD:D_Zener_Small_Filled
- R22, R24: footprint Resistor_SMD:R_0402_1005Metric -> OpenMD:R_0402_1005Metric; symbol Device:R_Small_US -> OpenMD:R_Small_US
- R23: footprint Resistor_SMD:R_2512_6332Metric -> OpenMD:R_2512_6332Metric; symbol Device:R_US -> OpenMD:R_US
- U8: footprint Package_TO_SOT_SMD:SOT-23-8 -> OpenMD:SOT-23-8; symbol Amplifier_Current:INA241A2xDDF -> OpenMD:INA241A2xDDF
Changed lines of the file:
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@@
 	(title_block
 		(title "Current Sense Amplifier")
-		(date "2024-05-19")
-		(rev "1")
+		(date "2024-12-19")
+		(rev "1.1")
 		(company "Crab Labs")
 		(comment 1 "Author: Orion Serup")
@@
 	)
 	(symbol
-		(lib_id "Device:C_Small")
+		(lib_id "OpenMD:C_Small")
 		(at 106.68 62.23 90)
 		(unit 1)
@@
 			)
 		)
-		(property "Footprint" "Capacitor_SMD:C_0402_1005Metric"
+		(property "Footprint" "OpenMD:C_0402_1005Metric"
 			(at 106.68 62.23 0)
 			(effects
@@
 	)
 	(symbol
-		(lib_id "Device:R_Small_US")
+		(lib_id "OpenMD:R_Small_US")
 		(at 101.6 55.88 0)
 		(unit 1)
@@
 			)
 		)
-		(property "Footprint" "Resistor_SMD:R_0402_1005Metric"
+		(property "Footprint" "OpenMD:R_0402_1005Metric"
 			(at 101.6 55.88 0)
 			(effects
@@
 	)
 	(symbol
-		(lib_id "Device:C_Small")
+		(lib_id "OpenMD:C_Small")
 		(at 87.63 83.82 0)
 		(unit 1)
@@
 			)
 		)
-		(property "Footprint" "Capacitor_SMD:C_0402_1005Metric"
+		(property "Footprint" "OpenMD:C_0402_1005Metric"
 			(at 87.63 83.82 0)
 			(effects
@@
 	)
 	(symbol
-		(lib_id "Device:R_US")
+		(lib_id "OpenMD:R_US")
 		(at 106.68 40.64 90)
 		(unit 1)
@@
 			)
 		)
-		(property "Footprint" "Resistor_SMD:R_2512_6332Metric"
+		(property "Footprint" "OpenMD:R_2512_6332Metric"
 			(at 106.934 39.624 90)
 			(effects
@@
 	)
 	(symbol
-		(lib_id "Device:R_Small_US")
+		(lib_id "OpenMD:R_Small_US")
 		(at 111.76 55.88 0)
 		(unit 1)
@@
 			)
 		)
-		(property "Footprint" "Resistor_SMD:R_0402_1005Metric"
+		(property "Footprint" "OpenMD:R_0402_1005Metric"
 			(at 111.76 55.88 0)
 			(effects
@@
 	)
 	(symbol
-		(lib_id "Device:D_Zener_Small_Filled")
+		(lib_id "OpenMD:D_Zener_Small_Filled")
 		(at 125.73 44.45 270)
 		(unit 1)
@@
 			)
 		)
-		(property "Footprint" "Diode_SMD:D_SOD-123F"
+		(property "Footprint" "OpenMD:D_SOD-123F"
 			(at 125.73 44.45 90)
 			(effects
@@
 	)
 	(symbol
-		(lib_id "Amplifier_Current:INA241A2xDDF")
+		(lib_id "OpenMD:INA241A2xDDF")
 		(at 106.68 81.28 90)
 		(mirror x)
@@
 			)
 		)
-		(property "Footprint" "Package_TO_SOT_SMD:SOT-23-8"
+		(property "Footprint" "OpenMD:SOT-23-8"
 			(at 123.19 81.28 0)
 			(effects
