File: GateDriver.kicad_sch (KiCad schematic)
At the start: 10 parts, among them U2 LM1205

Commit message: added more capacitance
Parts:
- C40, C41, C42: footprint Capacitor_SMD:C_0402_1005Metric -> OpenMD:C_0402_1005Metric; symbol Device:C -> OpenMD:C
- D13, D16: footprint Diode_SMD:D_0402_1005Metric -> OpenMD:D_0402_1005Metric; symbol Device:D_TVS_Small -> OpenMD:D_TVS_Small
- R6, R7, R8, R9: footprint Resistor_SMD:R_0402_1005Metric -> OpenMD:R_0402_1005Metric; symbol Device:R_US -> OpenMD:R_US
- U2: symbol uP1996:UP1966E -> OpenMD:UP1966E
Changed lines of the file:
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@@
 	(title_block
 		(title "Gate Driver")
-		(date "2024-05-19")
-		(rev "1")
+		(date "2024-12-19")
+		(rev "1.1")
 		(company "Crab Labs")
 		(comment 1 "Author: Orion Serup")
@@
 	)
 	(symbol
-		(lib_id "Device:D_TVS_Small")
+		(lib_id "OpenMD:D_TVS_Small")
 		(at 57.15 52.07 90)
 		(unit 1)
@@
 			)
 		)
-		(property "Footprint" "Diode_SMD:D_0402_1005Metric"
+		(property "Footprint" "OpenMD:D_0402_1005Metric"
 			(at 57.15 52.07 0)
 			(effects
@@
 	)
 	(symbol
-		(lib_id "Device:C")
+		(lib_id "OpenMD:C")
 		(at 176.53 66.04 180)
 		(unit 1)
@@
 			)
 		)
-		(property "Footprint" "Capacitor_SMD:C_0402_1005Metric"
+		(property "Footprint" "OpenMD:C_0402_1005Metric"
 			(at 175.5648 62.23 0)
 			(effects
@@
 	)
 	(symbol
-		(lib_id "Device:D_TVS_Small")
+		(lib_id "OpenMD:D_TVS_Small")
 		(at 43.18 52.07 90)
 		(unit 1)
@@
 			)
 		)
-		(property "Footprint" "Diode_SMD:D_0402_1005Metric"
+		(property "Footprint" "OpenMD:D_0402_1005Metric"
 			(at 43.18 52.07 0)
 			(effects
@@
 	)
 	(symbol
-		(lib_id "Device:R_US")
+		(lib_id "OpenMD:R_US")
 		(at 81.28 63.5 270)
 		(unit 1)
@@
 			)
 		)
-		(property "Footprint" "Resistor_SMD:R_0402_1005Metric"
+		(property "Footprint" "OpenMD:R_0402_1005Metric"
 			(at 81.026 64.516 90)
 			(effects
@@
 	)
 	(symbol
-		(lib_id "uP1996:UP1966E")
+		(lib_id "OpenMD:UP1966E")
 		(at 92.71 73.66 0)
 		(mirror x)
@@
 	)
 	(symbol
-		(lib_id "Device:C")
+		(lib_id "OpenMD:C")
 		(at 58.42 72.39 0)
 		(unit 1)
@@
 			)
 		)
-		(property "Footprint" "Capacitor_SMD:C_0402_1005Metric"
+		(property "Footprint" "OpenMD:C_0402_1005Metric"
 			(at 59.3852 76.2 0)
 			(effects
@@
 	)
 	(symbol
-		(lib_id "Device:R_US")
+		(lib_id "OpenMD:R_US")
 		(at 82.55 73.66 90)
 		(unit 1)
@@
 			)
 		)
-		(property "Footprint" "Resistor_SMD:R_0402_1005Metric"
+		(property "Footprint" "OpenMD:R_0402_1005Metric"
 			(at 82.804 72.644 90)
 			(effects
@@
 	)
 	(symbol
-		(lib_id "Device:R_US")
+		(lib_id "OpenMD:R_US")
 		(at 143.51 66.04 90)
 		(unit 1)
@@
 			)
 		)
-		(property "Footprint" "Resistor_SMD:R_0402_1005Metric"
+		(property "Footprint" "OpenMD:R_0402_1005Metric"
 			(at 143.764 65.024 90)
 			(effects
@@
 	)
 	(symbol
-		(lib_id "Device:C")
+		(lib_id "OpenMD:C")
 		(at 44.45 72.39 0)
 		(unit 1)
@@
 			)
 		)
-		(property "Footprint" "Capacitor_SMD:C_0402_1005Metric"
+		(property "Footprint" "OpenMD:C_0402_1005Metric"
 			(at 45.4152 76.2 0)
 			(effects
@@
 	)
 	(symbol
-		(lib_id "Device:R_US")
+		(lib_id "OpenMD:R_US")
 		(at 146.05 68.58 90)
 		(unit 1)
@@
 			)
 		)
-		(property "Footprint" "Resistor_SMD:R_0402_1005Metric"
+		(property "Footprint" "OpenMD:R_0402_1005Metric"
 			(at 146.304 67.564 90)
 			(effects

Commit message: fixes
Other:
- note added: "Substitute withh UP1966 or LT8418, same Footprint"
- note removed: "Substitute withh UP1966 or AD8418, same Footprint"
Changed lines of the file:
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@@
 		)
 	)
-	(text "Substitute withh UP1966 or AD8418, same Footprint\n"
+	(text "Substitute withh UP1966 or LT8418, same Footprint\n"
 		(exclude_from_sim no)
 		(at 109.982 44.958 0)
